File: Rev A/breaking_bitcoin.brd (EAGLE design)
At the start: 53.3 x 63.5 mm, 66 parts, among them J1 M20-9992046, J2 M20-9992046, J3 M20-9992046, J4 TC2050-IDC-NLFP, J5 DNP, J6 DNP, J7 ZX80-B-5P, Q1 DMG2302UK, U1 STM32F205RE, U2 MCP1703AT-3302E/CB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

Commit message: Improving 3.3V power plane
Routing:
- net 3.3V: track 46.0 -> 50.8 mm
Changed lines of the file:
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@@
 <setting verticaltext="up"/>
 </settings>
-<grid distance="50" unitdist="mil" unit="mil" style="lines" multiple="1" display="yes" altdistance="25" altunitdist="mil" altunit="mil"/>
+<grid distance="50" unitdist="mil" unit="mil" style="lines" multiple="1" display="yes" altdistance="5" altunitdist="mil" altunit="mil"/>
 <layers>
 <layer number="1" name="Top" color="4" fill="1" visible="yes" active="yes"/>
@@
 <via x="32.893" y="20.701" extent="1-16" drill="0.508"/>
 <wire x1="31.711" y1="19.812" x2="32.004" y2="19.812" width="0.3048" layer="16"/>
-<wire x1="32.004" y1="19.812" x2="32.893" y2="20.701" width="0.3048" layer="16"/>
+<wire x1="32.893" y1="20.701" x2="32.004" y2="19.812" width="0.3048" layer="16"/>
 <wire x1="32.17" y1="21.65" x2="32.17" y2="21.424" width="0.2921" layer="1"/>
 <wire x1="32.17" y1="21.424" x2="32.893" y2="20.701" width="0.2921" layer="1"/>
@@
 <wire x1="29.7279125" y1="21.336" x2="29.21" y2="21.336" width="0.2921" layer="1"/>
 <wire x1="30.41925" y1="20.6446625" x2="29.7279125" y2="21.336" width="0.2921" layer="1"/>
+<wire x1="32.893" y1="20.701" x2="33.528" y2="20.066" width="0.3048" layer="1"/>
+<wire x1="29.21" y1="21.336" x2="32.258" y2="21.336" width="0.3048" layer="16"/>
+<wire x1="32.258" y1="21.336" x2="32.893" y2="20.701" width="0.3048" layer="16"/>
 </signal>
 <signal name="VCORE">
