File: Rev A/breaking_bitcoin.sch (EAGLE design)
At the start: 66 parts, among them J1 M20-9992046, J2 M20-9992046, J3 M20-9992046, J4 TC2050-IDC-NLFP, J5 DNP, J6 M20-9990246, J7 ZX80-B-5P, Q1 DMG2302UK, U1 STM32F205RE, U2 MCP1703AT-3302E/CB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

Commit message: Adding BOM/Gerbers
Parts:
- C11, C12, C15, C17, C18, C19, C20, C21, C22, D3, J7, R10, R11, R12, R13, R14, R9, U2, U3, X1: NOTE (none) -> Trezor
- J6: value M20-9990246 -> DNP
- S1, S2: device SparkFun-Electromechanical:SWITCH-MOMENTARY-2PTH -> KVB-switches:SWITCH-TACT-TH; NOTE (none) -> Trezor
